Commit message: UR20 is attached onto a floating object to simulate the platform

File: mpc_simulation/mpc_description/urdf/ROS/ros_control.xacro (robot description, xacro)
@@ -7,4 +7,15 @@
     </plugin>
   </gazebo>
+  <transmission name="platform_x_trans">
+    <type>transmission_interface/SimpleTransmission</type>
+    <joint name="platform_x_joint">
+      <!-- Use PositionJointInterface to directly command position -->
+      <hardwareInterface>hardware_interface/PositionJointInterface</hardwareInterface>
+    </joint>
+    <actuator name="platform_x_motor">
+      <hardwareInterface>hardware_interface/PositionJointInterface</hardwareInterface>
+      <mechanicalReduction>1</mechanicalReduction>
+    </actuator>
+  </transmission>
 </xacro:macro>
 </robot>

File: mpc_simulation/mpc_description/urdf/mpc_robot.xacro (robot description, xacro)
@@ -11,6 +11,6 @@
   <!-- Include UR20 Arm -->
   <xacro:property name="arm_position_x" default="0.0"/>
-  <xacro:property name="arm_position_y" default="0.0"/>
-  <xacro:property name="arm_position_z" default="0.0"/>
+  <xacro:property name="arm_position_y" default="0.1"/>
+  <xacro:property name="arm_position_z" default="0.5"/>
   <xacro:property name="arm_orientation_r" default="0.0"/>
   <xacro:property name="arm_orientation_p" default="0.0"/>
@@ -27,5 +27,5 @@
       <joint name="base_joint" type="fixed">
         <origin xyz="${arm_position_x} ${arm_position_y} ${arm_position_z}" rpy="${arm_orientation_r} ${arm_orientation_p} ${arm_orientation_y}"/>
-        <parent link="world" />
+        <parent link="mobile_base_link" />
         <child link="base_link" />
       </joint>
@@ -37,7 +37,7 @@
       <joint name="base_joint" type="fixed">
         <origin xyz="${arm_position_x} ${arm_position_y} ${arm_position_z}" rpy="${arm_orientation_r} ${arm_orientation_p} ${arm_orientation_y}"/>
-        <parent link="world" />
+        <parent link="mobile_base_link" />
         <child link="base_link" />
-        </joint>
+      </joint>
     </xacro:unless>
     <joint name="tool_controller_fake_joint" type="fixed">
@@ -53,4 +53,22 @@
     <axis xyz="0 0 1" />
     </joint>
+    <link name="mobile_base_link">
+      <!-- Optional: Add minimal visual/collision/inertial properties if you want to see it or have it interact physically -->
+      <visual>
+        <geometry><box size="0.1 0.1 0.05"/></geometry>
+        <material name="grey"><color rgba="0.5 0.0 0.0 1"/></material>
+      </visual>
+      <inertial>
+        <mass value="1"/>
+        <inertia ixx="0.01" iyy="0.01" izz="0.01" ixy="0" ixz="0" iyz="0"/>
+      </inertial>
+    </link>
+    <joint name="platform_x_joint" type="prismatic">
+      <parent link="world"/>
+      <child link="mobile_base_link"/>
+      <origin xyz="0 0 0" rpy="0 0 0"/>
+      <axis xyz="1 0 0"/> <!-- Movement along X axis -->
+      <limit lower="-1.0" upper="1.0" effort="100" velocity="1.0"/> <!-- Adjust limits as needed -->
+    </joint>
   </xacro:macro>
   <xacro:mpc prefix="$(arg prefix)" load_kinematics_file="$(arg load_kinematics_file)"/>

Commit message: New naming convention

File: mpc_simulation/mpc_description/urdf/ROS/ros_control.xacro (robot description, xacro)
@@ -7,11 +7,11 @@
     </plugin>
   </gazebo>
-  <transmission name="platform_x_trans">
+  <transmission name="platform_prismatic_trans">
     <type>transmission_interface/SimpleTransmission</type>
-    <joint name="platform_x_joint">
+    <joint name="platform_prismatic_joint">
       <!-- Use VelocityJointInterface to directly command velocity -->
       <hardwareInterface>hardware_interface/VelocityJointInterface</hardwareInterface>
     </joint>
-    <actuator name="platform_x_motor">
+    <actuator name="platform_prismatic_motor">
       <hardwareInterface>hardware_interface/VelocityJointInterface</hardwareInterface>
       <mechanicalReduction>1</mechanicalReduction>

File: mpc_simulation/mpc_description/urdf/mpc_robot.xacro (robot description, xacro)
@@ -64,9 +64,9 @@
       </inertial>
     </link>
-    <joint name="platform_x_joint" type="prismatic">
+    <joint name="platform_prismatic_joint" type="prismatic">
       <parent link="world"/>
       <child link="mobile_base_link"/>
       <origin xyz="0 0 0" rpy="0 0 0"/>
-      <axis xyz="1 0 0"/> <!-- Movement along X axis -->
+      <axis xyz="0 1 0"/> <!-- Movement along X axis -->
       <limit lower="-1.0" upper="1.0" effort="100" velocity="1.0"/> <!-- Adjust limits as needed -->
     </joint>

Commit message: New configurable motion in simulation

File: mpc_simulation/mpc_description/urdf/ROS/ros_control.xacro (robot description, xacro)
@@ -1,21 +1,35 @@
 <?xml version="1.0"?>
 <robot xmlns:xacro="http://ros.org/wiki/xacro" name="arm_control">
-<xacro:macro name="ros_control" >
-  <gazebo>
-    <plugin name="gazebo_ros_control" filename="libgazebo_ros_control.so">
-      <robotNamespace>/</robotNamespace>
-    </plugin>
-  </gazebo>
-  <transmission name="platform_prismatic_trans">
-    <type>transmission_interface/SimpleTransmission</type>
-    <joint name="platform_prismatic_joint">
-      <!-- Use VelocityJointInterface to directly command velocity -->
-      <hardwareInterface>hardware_interface/VelocityJointInterface</hardwareInterface>
-    </joint>
-    <actuator name="platform_prismatic_motor">
-      <hardwareInterface>hardware_interface/VelocityJointInterface</hardwareInterface>
-      <mechanicalReduction>1</mechanicalReduction>
-    </actuator>
-  </transmission>
-</xacro:macro>
+  <xacro:arg name="motion_type" default="linear"/>
+  <xacro:macro name="ros_control" params="motion_type">
+    <gazebo>
+      <plugin name="gazebo_ros_control" filename="libgazebo_ros_control.so">
+        <robotNamespace>/</robotNamespace>
+      </plugin>
+    </gazebo>
+    <xacro:if value="${motion_type == 'linear'}">
+      <transmission name="platform_prismatic_trans">
+        <type>transmission_interface/SimpleTransmission</type>
+        <joint name="platform_prismatic_joint">
+          <hardwareInterface>hardware_interface/VelocityJointInterface</hardwareInterface>
+        </joint>
+        <actuator name="platform_prismatic_motor">
+          <hardwareInterface>hardware_interface/VelocityJointInterface</hardwareInterface>
+          <mechanicalReduction>1</mechanicalReduction>
+        </actuator>
+      </transmission>
+    </xacro:if>
+    <xacro:if value="${motion_type == 'angular'}">
+      <transmission name="platform_revolute_trans">
+        <type>transmission_interface/SimpleTransmission</type>
+        <joint name="platform_revolute_joint">
+          <hardwareInterface>hardware_interface/VelocityJointInterface</hardwareInterface>
+        </joint>
+        <actuator name="platform_revolute_motor">
+          <hardwareInterface>hardware_interface/VelocityJointInterface</hardwareInterface>
+          <mechanicalReduction>1</mechanicalReduction>
+        </actuator>
+      </transmission>
+    </xacro:if>
+  </xacro:macro>
 </robot>

File: mpc_simulation/mpc_description/urdf/mpc_robot.xacro (robot description, xacro)
@@ -16,7 +16,9 @@
   <xacro:property name="arm_orientation_p" default="0.0"/>
   <xacro:property name="arm_orientation_y" default="0.0"/>
+  <!-- Arguments -->
   <xacro:arg name="prefix" default="" />
   <xacro:arg name="load_kinematics_file" default="true"/>
-  <xacro:macro name="mpc" params="prefix load_kinematics_file">
+  <xacro:arg name="motion_type" default="linear"/>
+  <xacro:macro name="mpc" params="prefix load_kinematics_file motion_type">
     <link name="world" />
     <!-- UR20 Robot Arm    -->
@@ -64,14 +66,26 @@
       </inertial>
     </link>
-    <joint name="platform_prismatic_joint" type="prismatic">
-      <parent link="world"/>
-      <child link="mobile_base_link"/>
-      <origin xyz="0 0 0" rpy="0 0 0"/>
-      <axis xyz="0 1 0"/> <!-- Movement along X axis -->
-      <limit lower="-1.0" upper="1.0" effort="100" velocity="1.0"/> <!-- Adjust limits as needed -->
-    </joint>
+    <!-- Conditional Joint Definition based on motion_type -->
+    <xacro:if value="${motion_type == 'linear'}">
+      <joint name="platform_prismatic_joint" type="prismatic">
+        <parent link="world"/>
+        <child link="mobile_base_link"/>
+        <origin xyz="0 0 0" rpy="0 0 0"/>
+        <axis xyz="0 1 0"/> <!-- Defaulting to Y axis for linear motion -->
+        <limit lower="-1.0" upper="1.0" effort="100" velocity="1.0"/>
+      </joint>
+    </xacro:if>
+    <xacro:if value="${motion_type == 'angular'}">
+      <joint name="platform_revolute_joint" type="revolute">
+        <parent link="world"/>
+        <child link="mobile_base_link"/>
+        <origin xyz="0 0 0" rpy="0 0 0"/>
+        <axis xyz="0 0 1"/> <!-- Rotation around Z axis -->
+        <limit lower="-${pi}" upper="${pi}" effort="100" velocity="1.0"/>
+      </joint>
+    </xacro:if>
   </xacro:macro>
-  <xacro:mpc prefix="$(arg prefix)" load_kinematics_file="$(arg load_kinematics_file)"/>
-  <xacro:ros_control/>
+  <xacro:mpc prefix="$(arg prefix)" load_kinematics_file="$(arg load_kinematics_file)" motion_type="$(arg motion_type)"/>
+  <xacro:ros_control motion_type="$(arg motion_type)"/>
   <!-- Add Gazebo plugin to publish ground truth odometry for mobile_base_link -->
   <gazebo>
