Commit message: Complex Dynamic Model created for mobile platform

File: mpc_simulation/mpc_description/urdf/mpc_robot.xacro (robot description, xacro)
@@ -72,5 +72,5 @@
         <child link="mobile_base_link"/>
         <origin xyz="0 0 0" rpy="0 0 0"/>
-        <axis xyz="0 1 0"/> <!-- Defaulting to Y axis for linear motion -->
+        <axis xyz="1 0 0"/> <!-- Defaulting to Y axis for linear motion -->
         <limit lower="-1.0" upper="1.0" effort="100" velocity="1.0"/>
       </joint>
